File: PCB/Circuit.kicad_sch (KiCad schematic)
At the start: 7 parts, among them J1 AudioJack4, SW1 SW_Push, SW2 SW_Push, SW3 SW_Push, U1 OLED Screen

Commit message: Add files via upload
Parts:
- added Li-Ion: Battery_Cell, symbol Device:Battery_Cell
- added R1: 1k, symbol Device:R
- added R2: 680, symbol Device:R
- added U2: MT3608, Package_TO_SOT_SMD:SOT-23-6, symbol Regulator_Switching:MT3608
- added U3: TP4057, Package_TO_SOT_SMD:TSOT-23-6, symbol Battery_Management:TP4057
Connections:
- net GND: now also R1.2, U2.3 (FB)
- net at SW1.1: now also A1.8 (D5); no longer A1.7 (D4)
- net at SW2.1: now also A1.10 (D7); no longer A1.9 (D6)
- net at DFPLAYER MINI1.2 (RX): now also R1.1, R2.2; no longer A1.5 (D2)
- net at DFPLAYER MINI1.3 (TX): now also A1.6 (D3); no longer A1.2 (D0/RX)
- net at A1.11 (D8): no longer SW3.1
- net at A1.12 (D9): now also SW3.1
- net +5V renamed VCC
- net VCC: now also U2.1 (SW)
- net +9V: no longer names the net of A1.30 (VIN)
- new net: U2.5 (IN), U3.2 (GND)
- new net: Li-Ion.2 (-), U3.3 (BAT)
- new net: U2.4 (EN), U3.4 (V_{CC})
- new net: Li-Ion.1 (+), U3.6 (PROG)
- new net: A1.5 (D2), R2.1
Other:
- note added: "B+"
- note added: "B-"
- note added: "Battery Management"
- note added: "IN+"
- note added: "IN-"
- note added: "OUT+"
- note added: "OUT-"

Commit message: Add files via upload
Parts:
- added SW4: SW_DPST_x2, symbol Switch:SW_DPST_x2
Connections:
- net at U3.2 (GND): now also SW4.1 (A); no longer U2.5 (IN)
- new net: SW4.2 (B), U2.5 (IN)
Changed lines of the file:
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@@
 	)
 	(rectangle
-		(start 22.86 78.74)
+		(start 22.86 77.47)
 		(end 102.87 99.06)
 		(stroke
@@
 		)
 	)
+	(text "Left Button"
+		(exclude_from_sim no)
+		(at 61.214 53.34 0)
+		(effects
+			(font
+				(size 1.016 1.016)
+			)
+		)
+	)
+	(text "OUT+\n"
+		(exclude_from_sim no)
+		(at 34.29 85.598 0)
+		(effects
+			(font
+				(size 1.27 1.27)
+			)
+		)
+	)
+	(text "OUT-"
+		(exclude_from_sim no)
+		(at 34.544 92.964 0)
+		(effects
+			(font
+				(size 1.27 1.27)
+			)
+		)
+	)
 	(text "Right Button"
 		(exclude_from_sim no)
-		(at 61.722 53.34 0)
-		(effects
-			(font
-				(size 1.016 1.016)
-			)
-		)
-	)
-	(text "OUT+\n"
-		(exclude_from_sim no)
-		(at 34.29 85.598 0)
-		(effects
-			(font
-				(size 1.27 1.27)
-			)
-		)
-	)
-	(text "OUT-"
-		(exclude_from_sim no)
-		(at 34.544 92.964 0)
-		(effects
-			(font
-				(size 1.27 1.27)
-			)
-		)
-	)
-	(text "Left Button"
-		(exclude_from_sim no)
-		(at 61.214 43.18 0)
+		(at 61.722 43.18 0)
 		(effects
 			(font
@@
 	(wire
 		(pts
+			(xy 62.23 81.28) (xy 80.01 81.28)
+		)
+		(stroke
+			(width 0)
+			(type default)
+		)
+	)
+	(wire
+		(pts
 			(xy 44.45 85.09) (xy 44.45 86.36)
 		)
@@
 	(wire
 		(pts
-			(xy 34.29 81.28) (xy 80.01 81.28)
+			(xy 34.29 81.28) (xy 52.07 81.28)
 		)
 		(stroke
@@
 					(unit 1)
 				)
+			)
+		)
+	)
+	(symbol
+		(lib_id "Switch:SW_DPST_x2")
+		(at 57.15 81.28 0)
+		(unit 1)
+		(body_style 1)
+		(exclude_from_sim no)
+		(in_bom yes)
+		(on_board yes)
+		(in_pos_files yes)
+		(dnp no)
+		(fields_autoplaced yes)
+		(property "Reference" "SW4"
+			(at 57.15 74.93 0)
+			(hide yes)
+			(show_name no)
+			(do_not_autoplace no)
+			(effects
+				(font
+					(size 1.27 1.27)
+				)
+			)
+		)
+		(property "Value" "SW_DPST_x2"
+			(at 57.15 77.47 0)
+			(hide yes)
+			(show_name no)
+			(do_not_autoplace no)
+			(effects
+				(font
+					(size 1.27 1.27)
+				)
+			)
+		)
+		(property "Footprint" ""
+			(at 57.15 81.28 0)
+			(hide yes)
+			(show_name no)
+			(do_not_autoplace no)
+			(effects
+				(font
+					(size 1.27 1.27)
+				)
+			)
+		)
+		(property "Datasheet" ""
+			(at 57.15 81.28 0)
+			(hide yes)
+			(show_name no)
+			(do_not_autoplace no)
+			(effects
+				(font
+					(size 1.27 1.27)
+				)
+			)
+		)
+		(property "Description" "Single Pole Single Throw (SPST) switch, separate symbol"
+			(at 57.15 81.28 0)
+			(hide yes)
+			(show_name no)
+			(do_not_autoplace no)
+			(effects
+				(font
+					(size 1.27 1.27)
+				)
+			)
+		)
+		(pin "1"
+		)
+		(pin "3"
+		)
+		(pin "2"
+		)
+		(pin "4"
+		)
+		(instances
+			(project "Circuit"
+				(path "/85cf9c24-144f-4343-ae5b-81f014581756"
+					(reference "SW4")
+					(unit 1)
+				)
